File: hardware/hardware.sch (KiCad schematic (older format))
At the start: 5 parts, among them P1 Conn_02x20_Odd_Even

Commit message: Added the ATMega328p and a 8MHz crystal
Parts:
- removed MK1, MK2, MK3, MK4: M2.5, MountingHole:MountingHole_2.7mm_M2.5, symbol hardware-rescue:Mounting_Hole-Mechanical
- added C? (x2): 22p, symbol Device:C
- added MK1, MK2, MK3, MK4: 2.5, symbol Hardware:MOUNTING_HOLE
- added U?: ATmega328P-AU, Package_QFP:TQFP-32_7x7mm_P0.8mm, symbol MCU_Microchip_ATmega:ATmega328P-AU
- added Y?: 8MHz, symbol Device:Crystal
Connections:
- net labels added: +3V, PB0, PB1, PB2, PB3, PB4, PB5, PB6(XTAL1), PB7(XTAL2), PC0, PC1, PC2, PC3, PC4, PC5, PC6, PD0, PD1, PD2, PD3, PD4, PD5, PD6, PD7
- net labels removed: +3.3V
- wire segments 52 -> 90
